Commit message: Fix moodel called bug

File: dev_ws/src/robot_description/urdf/robot.urdf.xacro (robot description, xacro)
@@ -1,4 +1,4 @@
 <?xml version="1.0"?>
-<robot name="durian_robot" xmlns:xacro="http://www.ros.org">
+<robot name="durian_robot" xmlns:xacro="http://www.ros.org/wiki/xacro">
     <!-- Core -->
     <xacro:include filename="$(find robot_description)/urdf/robot_core.xacro"/>
@@ -6,27 +6,4 @@
     <xacro:include filename="$(find robot_description)/urdf/robot_sensor.xacro"/>
     <!-- Gazebo -->
-    <xacro:include filename="$(find robot_description)/urdf/robot_gazebo.xacro"/>
+    <!-- <xacro:include filename="$(find robot_description)/urdf/robot_gazebo.xacro"/> -->
 </robot>
-    <!-- <link name="base_link">
-        <visual>
-            <origin xyz="-0.0 0 -0.0" rpy="0 0 0"/>
-            <geometry>
-                <mesh filename="file://$(find robot_description)/meshes/robot.dae" scale="1 1 1"/>
-            </geometry>
-            <material name="Orange">
-            <color rgba="1.0 0.5 0 1.0"/>
-            </material>
-        </visual>
-        <collision>
-        <origin xyz="-0.0 0 -0.0" rpy="0 0 0"/>
-            <geometry>
-                <mesh filename="file://$(find robot_description)/meshes/robot.dae" scale="1 1 1"/>
-            </geometry>
-        </collision>
-        <inertial>
-        <origin xyz="0 0 -0.75" rpy="0 0 0"/>
-            <mass value="2000.0"/>
-             <inertia ixx="2800.3" ixy="0.0" ixz="0.0" iyy="2800.6" iyz="0.0" izz="1500.8" />
-            <!-- <inertia ixx="0.163" ixy="0.1" ixz="0.1" iyy="0.163" iyz="0.1" izz="0.163" /> -->
-        </inertial>
-    </link> -->

File: dev_ws/src/robot_description/urdf/robot_core.xacro (robot description, xacro)
@@ -1,11 +1,12 @@
 <?xml version="1.0"?>
 <robot xmlns:xacro="http://www.ros.org/wiki/xacro" >
-    <xacro:include filename="inertial_macros.xacro"/>
-    <xacro:include filename="robot_type.xacro"/>
+    <!-- Include xacro -->
+    <xacro:include filename="$(find robot_description)/urdf/robot_type.xacro"/>
+    <!-- Base structure -->
     <link name="base_link">
         <visual>
-            <origin xyz="-0.0 0 0.06" rpy="0 0 0"/>
+            <origin xyz="0 0 0" rpy="0 0 0"/>
             <geometry>
-                <mesh filename="file://$(find robot_description)/meshes/base.dae" scale="1 1 1"/>
+                <box size="0.6 0.6 0.3"/>
             </geometry>
             <material name="Orange">
@@ -14,18 +15,14 @@
         </visual>
         <collision>
-            <origin xyz="-0.0 0 0.06" rpy="0 0 0"/>
+            <origin xyz="0 0 0" rpy="0 0 0"/>
             <geometry>
-                <mesh filename="file://$(find robot_description)/meshes/base.dae" scale="1 1 1"/>
+                <box size="0.6 0.6 0.3"/>
             </geometry>
         </collision>
-        <!-- <inertial>
-            <origin xyz="0 0 -0.75" rpy="0 0 0"/>
-            <mass value="2000.0"/>
-            <inertia ixx="2800.3" ixy="0.0" ixz="0.0" iyy="2800.6" iyz="0.0" izz="1500.8"/>
-        </inertial> -->
     </link>
-    <xacro:wheel num="1" pos_x="0.1" pos_y="0.3" pos_z="0.06"/>
-    <xacro:wheel num="2" pos_x="-0.1" pos_y="0.3" pos_z="0.06"/>
-    <xacro:wheel num="3" pos_x="0.1" pos_y="-0.3" pos_z="0.06"/>
-    <xacro:wheel num="4" pos_x="-0.1" pos_y="-0.3" pos_z="0.06"/>
+    <!-- Wheel -->
+    <xacro:wheel number="1" pos_x="0.35" pos_y="0.2" pos_z="0"/>
+    <xacro:wheel number="2" pos_x="-0.35" pos_y="0.2" pos_z="0"/>
+    <xacro:wheel number="3" pos_x="0.35" pos_y="-0.2" pos_z="0"/>
+    <xacro:wheel number="4" pos_x="-0.35" pos_y="-0.2" pos_z="0"/>
 </robot>

File: dev_ws/src/robot_description/urdf/robot_type.xacro (robot description, xacro)
@@ -1,15 +1,17 @@
 <?xml version="1.0"?>
-<robot xmlns:xacro="http://ros.org/wiki/xacro">
-  <xacro:macro name="wheel" params="num pos_x pos_y pos_z">
-    <joint name="type_joint_${num}" type="continuous">
+<robot xmlns:xacro="http://www.ros.org/wiki/xacro">
+  <xacro:macro name="wheel" number="" pos_x="" pos_y="" pos_z="">
+    <!-- Joint -->
+    <joint name="type_joint_${number}" type="continuous">
       <parent link="base_link"/>
-      <child link="type_link_${num}"/>
+      <child link="type_link_${number}"/>
       <origin xyz="${pos_x} ${pos_y} ${pos_z}" rpy="0 0 0"/>
     </joint>
-    <link name="type_link_${num}">
+    <!-- Link -->
+    <link name="type_link_${number}">
       <visual>
         <origin xyz="0 0 0" rpy="0 0 0"/>
         <geometry>
-          <mesh filename="file://$(find robot_description)/meshes/type.dae" scale="1 1 1"/>
+          <cylinder radius="0.1" length="0.1"/>
         </geometry>
         <material name="Blue">
@@ -20,5 +22,5 @@
         <origin xyz="0 0 0" rpy="0 0 0"/>
         <geometry>
-          <mesh filename="file://$(find robot_description)/meshes/type.dae" scale="1 1 1"/>
+          <cylinder radius="0.1" length="0.1"/>
         </geometry>
       </collision>

Commit message: Add and fix bug control joint gz sim

File: dev_ws/src/robot_description/urdf/robot.urdf.xacro (robot description, xacro)
@@ -3,7 +3,5 @@
     <!-- Core -->
     <xacro:include filename="$(find robot_description)/urdf/robot_core.xacro"/>
-    <!-- Sensor -->
-    <xacro:include filename="$(find robot_description)/urdf/robot_sensor.xacro"/>
     <!-- Gazebo -->
-    <!-- <xacro:include filename="$(find robot_description)/urdf/robot_gazebo.xacro"/> -->
+    <xacro:include filename="$(find robot_description)/urdf/robot_gazebo.xacro"/>
 </robot>

File: dev_ws/src/robot_description/urdf/robot_core.xacro (robot description, xacro)
@@ -5,24 +5,31 @@
     <!-- Base structure -->
     <link name="base_link">
-        <visual>
-            <origin xyz="0 0 0" rpy="0 0 0"/>
-            <geometry>
-                <box size="0.6 0.6 0.3"/>
-            </geometry>
-            <material name="Orange">
-                <color rgba="1.0 0.5 0 1.0"/>
-            </material>
-        </visual>
-        <collision>
-            <origin xyz="0 0 0" rpy="0 0 0"/>
-            <geometry>
-                <box size="0.6 0.6 0.3"/>
-            </geometry>
-        </collision>
+      <visual>
+        <origin xyz="0 0 0" rpy="0 0 0"/>
+        <geometry>
+          <box size="0.6 0.6 0.3"/>
+        </geometry>
+        <material name="Orange">
+          <color rgba="1.0 0.5 0 1.0"/>
+        </material>
+      </visual>
+      <collision>
+        <origin xyz="0 0 0" rpy="0 0 0"/>
+        <geometry>
+          <box size="0.6 0.6 0.3"/>
+        </geometry>
+      </collision>
+      <inertial>
+        <mass value="5.0"/>
+        <origin xyz="0 0 0" rpy="0 0 0"/>
+        <inertia ixx="0.1" ixy="0.0" ixz="0.0"
+                 iyy="0.1" iyz="0.0"
+                 izz="0.1"/>
+      </inertial>
     </link>
     <!-- Wheel -->
-    <xacro:wheel number="1" pos_x="0.35" pos_y="0.2" pos_z="0"/>
-    <xacro:wheel number="2" pos_x="-0.35" pos_y="0.2" pos_z="0"/>
-    <xacro:wheel number="3" pos_x="0.35" pos_y="-0.2" pos_z="0"/>
-    <xacro:wheel number="4" pos_x="-0.35" pos_y="-0.2" pos_z="0"/>
+    <xacro:wheel number="1" pos_x="0.40" pos_y="0.25" pos_z="-0.2"/>
+    <xacro:wheel number="2" pos_x="-0.40" pos_y="0.25" pos_z="-0.2"/>
+    <xacro:wheel number="3" pos_x="0.40" pos_y="-0.25" pos_z="-0.2"/>
+    <xacro:wheel number="4" pos_x="-0.40" pos_y="-0.25" pos_z="-0.2"/>
 </robot>

File: dev_ws/src/robot_description/urdf/robot_sensor.xacro (robot description, xacro)
@@ -1,3 +1,47 @@
 <?xml version="1.0"?>
 <robot xmlns:xacro="http://www.ros.org/wiki/xacro">
+  <!-- Camera link -->
+  <link name="camera_link">
+    <visual>
+      <geometry>
+        <box size="0.1 0.1 0.1"/>
+      </geometry>
+    </visual>
+    <collision>
+      <geometry>
+        <box size="0.1 0.1 0.1"/>
+      </geometry>
+    </collision>
+    <inertial>
+      <mass value="0.0001"/>
+        <inertia ixx="0.1" ixy="0" ixz="0" iyy="0.1" iyz="0" izz="0.1" />
+    </inertial>
+  </link>
+  <!-- Camera joint -->
+  <joint name="camera_joint" type="fixed">
+    <parent link="base_link"/>
+    <child link="camera_link"/>
+    <origin xyz="0 0 0.4" rpy="0 -1.57 0"/>
+  </joint>
+  <!-- Camera sensor -->
+  <gazebo reference="camera_link">
+    <sensor name="front_cam" type="camera">
+      <gz_frame_id>base_link</gz_frame_id>
+      <camera>
+        <horizontal_fov>1.047</horizontal_fov>
+        <image>
+          <width>1920</width>
+          <height>1080</height>
+        </image>
+        <clip>
+          <near>0.1</near>
+          <far>100</far>
+        </clip>
+      </camera>
+      <always_on>1</always_on>
+      <update_rate>30</update_rate>
+      <visualize>true</visualize>
+      <topic>camera_up</topic>
+    </sensor>
+  </gazebo>
 </robot>

File: dev_ws/src/robot_description/urdf/robot_type.xacro (robot description, xacro)
@@ -1,13 +1,15 @@
 <?xml version="1.0"?>
 <robot xmlns:xacro="http://www.ros.org/wiki/xacro">
-  <xacro:macro name="wheel" number="" pos_x="" pos_y="" pos_z="">
+  <xacro:macro name="wheel" params="number pos_x pos_y pos_z">
     <!-- Joint -->
-    <joint name="type_joint_${number}" type="continuous">
+    <joint name="wheel_${number}_joint" type="continuous">
       <parent link="base_link"/>
-      <child link="type_link_${number}"/>
-      <origin xyz="${pos_x} ${pos_y} ${pos_z}" rpy="0 0 0"/>
+      <child link="wheel_${number}_link"/>
+      <axis xyz="0 0 1"/>
+      <origin xyz="${pos_x} ${pos_y} ${pos_z}" rpy="-1.57 0 0"/>
+      <limit effort="100.0" velocity="20.0" lower="-3.14" upper="3.14"/>
     </joint>
     <!-- Link -->
-    <link name="type_link_${number}">
+    <link name="wheel_${number}_link">
       <visual>
         <origin xyz="0 0 0" rpy="0 0 0"/>
@@ -27,6 +29,6 @@
       <inertial>
         <origin xyz="0 0 0" rpy="0 0 0"/>
-        <mass value="100.0"/>
-        <inertia ixx="10.0" ixy="0.0" ixz="0.0" iyy="10.0" iyz="0.0" izz="10.0"/>
+        <mass value="1.0"/>
+        <inertia ixx="0.01" ixy="0.0" ixz="0.0" iyy="0.01" iyz="0.0" izz="0.01"/>
       </inertial>
     </link>

Commit message: Add kinematic to point by IMU

File: dev_ws/src/robot_description/urdf/robot.urdf.xacro (robot description, xacro)
@@ -5,3 +5,5 @@
     <!-- Gazebo -->
     <xacro:include filename="$(find robot_description)/urdf/robot_gazebo.xacro"/>
+    <!-- Sensors -->
+    <xacro:include filename="$(find robot_description)/urdf/robot_sensor.xacro"/>
 </robot>

File: dev_ws/src/robot_description/urdf/robot_core.xacro (robot description, xacro)
@@ -2,4 +2,5 @@
 <robot xmlns:xacro="http://www.ros.org/wiki/xacro" >
     <!-- Include xacro -->
+    <xacro:include filename="$(find robot_description)/urdf/robot_steering.xacro"/>
     <xacro:include filename="$(find robot_description)/urdf/robot_type.xacro"/>
     <!-- Base structure -->
@@ -8,5 +9,5 @@
         <origin xyz="0 0 0" rpy="0 0 0"/>
         <geometry>
-          <box size="0.6 0.6 0.3"/>
+          <box size="1 1 0.3"/> <!-- z: -0.15 -->
         </geometry>
         <material name="Orange">
@@ -17,5 +18,5 @@
         <origin xyz="0 0 0" rpy="0 0 0"/>
         <geometry>
-          <box size="0.6 0.6 0.3"/>
+          <box size="1 1 0.3"/>
         </geometry>
       </collision>
@@ -29,7 +30,7 @@
     </link>
     <!-- Wheel -->
-    <xacro:wheel number="1" pos_x="0.40" pos_y="0.25" pos_z="-0.2"/>
-    <xacro:wheel number="2" pos_x="-0.40" pos_y="0.25" pos_z="-0.2"/>
-    <xacro:wheel number="3" pos_x="0.40" pos_y="-0.25" pos_z="-0.2"/>
-    <xacro:wheel number="4" pos_x="-0.40" pos_y="-0.25" pos_z="-0.2"/>
+    <xacro:wheel prefix="steering_1_link" number="1" pos_x="0" pos_y="0.075" pos_z="-0.075"/>
+    <xacro:wheel prefix="steering_2_link" number="2" pos_x="0" pos_y="0.075" pos_z="-0.075"/>
+    <xacro:wheel prefix="steering_3_link" number="3" pos_x="0" pos_y="-0.075" pos_z="-0.075"/>
+    <xacro:wheel prefix="steering_4_link" number="4" pos_x="0" pos_y="-0.075" pos_z="-0.075"/>
 </robot>

File: dev_ws/src/robot_description/urdf/robot_gazebo.xacro (robot description, xacro)
@@ -30,4 +30,24 @@
       <topic>/wheel_4_joint/command</topic>
     </plugin>
+    <plugin filename="gz-sim-joint-controller-system" name="gz::sim::systems::JointController">
+      <joint_name>steering_1_joint</joint_name>
+      <use_force_commands>true</use_force_commands>
+      <topic>/steering_1_joint/command</topic>
+    </plugin>
+    <plugin filename="gz-sim-joint-controller-system" name="gz::sim::systems::JointController">
+      <joint_name>steering_2_joint</joint_name>
+      <use_force_commands>true</use_force_commands>
+      <topic>/steering_2_joint/command</topic>
+    </plugin>
+    <plugin filename="gz-sim-joint-controller-system" name="gz::sim::systems::JointController">
+      <joint_name>steering_3_joint</joint_name>
+      <use_force_commands>true</use_force_commands>
+      <topic>/steering_3_joint/command</topic>
+    </plugin>
+    <plugin filename="gz-sim-joint-controller-system" name="gz::sim::systems::JointController">
+      <joint_name>steering_4_joint</joint_name>
+      <use_force_commands>true</use_force_commands>
+      <topic>/steering_4_joint/command</topic>
+    </plugin>
     <plugin filename="gz-sim-joint-state-publisher-system" name="gz::sim::systems::JointStatePublisher">
       <topic>joint_states</topic>
@@ -36,4 +56,8 @@
       <joint_name>wheel_3_joint</joint_name>
       <joint_name>wheel_4_joint</joint_name>
+      <joint_name>steering_1_joint</joint_name>
+      <joint_name>steering_2_joint</joint_name>
+      <joint_name>steering_3_joint</joint_name>
+      <joint_name>steering_4_joint</joint_name>
     </plugin>
   </gazebo>

File: dev_ws/src/robot_description/urdf/robot_sensor.xacro (robot description, xacro)
@@ -1,4 +1,14 @@
 <?xml version="1.0"?>
 <robot xmlns:xacro="http://www.ros.org/wiki/xacro">
+  <!-- IMU -->
+  <gazebo reference="base_link">
+      <sensor name="imu_sensor" type="imu">
+          <pose relative_to="base_link">0 0 0 0 0 0</pose>
+          <always_on>1</always_on>
+          <update_rate>1000.0</update_rate>
+          <topic>imu</topic>
+          <gz_frame_id>base_link</gz_frame_id>
+      </sensor>
+  </gazebo>
   <!-- Camera link -->
   <link name="camera_link">

File: dev_ws/src/robot_description/urdf/robot_type.xacro (robot description, xacro)
@@ -1,8 +1,8 @@
 <?xml version="1.0"?>
 <robot xmlns:xacro="http://www.ros.org/wiki/xacro">
-  <xacro:macro name="wheel" params="number pos_x pos_y pos_z">
+  <xacro:macro name="wheel" params="prefix number pos_x pos_y pos_z">
     <!-- Joint -->
     <joint name="wheel_${number}_joint" type="continuous">
-      <parent link="base_link"/>
+      <parent link="${prefix}"/>
       <child link="wheel_${number}_link"/>
       <axis xyz="0 0 1"/>
